File: Hardware/DAQ.sch (EAGLE design)
At the start: 35 parts, among them U1 DAC8564IAPW, U2 AD7606BSTZ

Commit message: added usart interface
Parts:
- removed AUX, CHANNEL_X, CHANNEL_Y, CHANNEL_Z: 1-227161-0, con-coax:1-227161-0
- removed JP1: (no value), pinhead:PINHD-1X8
- removed JP4: (no value), pinhead:PINHD-1X4
- added C16, C17, C18: (no value), resistor:C-EUC0805
- added IC2: FT232RL, ftdichip:FT232RL
- added JP3: (no value), pinhead:PINHD-1X8
- added X1: PN61729-S, con-berg:PN61729-S
- C10, C8, C9: device resistor:CPOL-EUE5-8.5 -> resistor:C-EUC0805K
Connections:
- removed net AGND: C1.2, C10.-, C2.2, C3.2, C4.2, C5.2, C6.2, C7.2, C8.-, C9.-, JP4.1, JP4.2, JP4.3, JP4.4, U2.AGND_10, U2.AGND_11, U2.AGND_14, U2.AGND_2, U2.AGND_4, U2.AGND_5, U2.AGND_6, U2.AGND_7, U2.AGND_8, U2.AGND_9, U2.DB0, U2.DB1, U2.DB10, U2.DB11, U2.DB12, U2.DB13, U2.DB15/BYTE_SEL, U2.DB2, U2.DB3, U2.DB4, U2.DB5, U2.DB6, U2.DB9, U2.OS_0, U2.OS_1, U2.RANGE, U2.REFGND, U2.REFGND_2, U2.V1GND, U2.V2GND, U2.V3GND, U2.V4GND
- removed net N$12: JP1.2, U2.V2
- removed net N$13: JP1.5, U2.V3
- removed net N$14: JP1.6, U2.V4
- removed net N$4: JP1.3, U2.AGND
- removed net SP1_SCLK: JP2.3, U2.~RD/SCLK
- net GND: now also C1.2, C10.2, C16.2, C17.2, C18.2, C2.2, C3.2, C4.2, C5.2, C6.2, C7.2, C8.2, C9.2, IC2.GND, IC2.GND@1, IC2.GND@2, IC2.GND@A, IC2.TEST, JP3.2, JP3.4, JP3.6, JP3.8, U2.AGND_10, U2.AGND_11, U2.AGND_14, U2.AGND_2, U2.AGND_4, U2.AGND_5, U2.AGND_6, U2.AGND_7, U2.AGND_8, U2.AGND_9, U2.DB0, U2.DB1, U2.DB10, U2.DB11, U2.DB12, U2.DB13, U2.DB15/BYTE_SEL, U2.DB2, U2.DB3, U2.DB4, U2.DB5, U2.DB6, U2.DB9, U2.OS_0, U2.OS_1, U2.RANGE, U2.REFGND, U2.REFGND_2, U2.V1GND, U2.V2GND, U2.V3GND, U2.V4GND, X1.4, X1.S1, X1.S2; no longer AUX.2, CHANNEL_X.2, CHANNEL_Y.2, CHANNEL_Z.2
- net N$1: now also C16.1, C18.1, IC2.VCC, X1.1; no longer JP1.8, U2.AGND_3
- net N$11: now also C17.1, IC2.3V3OUT, IC2.VCCIO; no longer JP1.1, U2.V1
- net N$15: now also C10.1; no longer C10.+
- net N$19: now also JP3.1; no longer CHANNEL_X.1
- net N$2: now also IC2.USBDM, X1.2; no longer JP1.4, U2.AGND_12
- net N$21: now also JP3.3; no longer CHANNEL_Y.1
- net N$23: now also JP3.5; no longer CHANNEL_Z.1
- net N$25: now also JP3.7; no longer AUX.1
- net N$3: now also IC2.USBDP, X1.3; no longer JP1.7, U2.AGND_13
- net N$8: now also C8.1; no longer C8.+
- net N$9: now also C9.1; no longer C9.+
- net Q1-Q2_BUF: now also U2.V1
- net Q1-Q4_BUF: now also U2.AGND
- net Q1_BUF: now also U2.AGND_12
- net Q2-Q3_BUF: now also U2.AGND_3
- net Q2_BUF: now also U2.V3
- net Q3_BUF: now also U2.V4
- net Q4-Q3_BUF: now also U2.V2
- net Q4_BUF: now also U2.AGND_13
- net SPI1_SCLK: now also JP2.3, U2.~RD/SCLK
- net USART3_RX: now also IC2.TXD
- net USART3_TX: now also IC2.RXD
Other:
- moved on the sheet: X2-1, X2-10, X2-11, X2-12, X2-13, X2-14, X2-15, X2-2, X2-3, X2-4, X2-5, X2-6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

Commit message: finished board layout
Parts:
- removed JP2: (no value), pinhead:PINHD-1X8
- added C19, C20, C21, C22, C23, C24, C25, C26: (no value), resistor:C-EUC0805K
- added D1: 1N4004, diode:1N4004
- added IC3, IC4, IC5: MCP1703DB, linear:MCP1703DB
- added JP1: (no value), pinhead:PINHD-1X2
- added JP4: (no value), pinhead:PINHD-1X3
- C13, C14: device resistor:CPOL-EUE5-6 -> resistor:C-EUC0805
Connections:
- new net N$12: C21.1, IC5.VO, JP1.1
- new net N$29: C22.1, C23.1, C24.1, D1.C, IC3.VI, IC4.VI, IC5.VI
- net +15V: now also C25.1, D1.A, IC1P.V+, JP4.1
- net +3V3: now also C13.1, C14.1, C20.1, IC3.VO; no longer C13.+, C14.+, JP2.8
- net +5V: now also C19.1, IC4.VO; no longer JP2.7
- net -15V: now also C26.1, IC1P.V-, JP4.3
- net BUSY: no longer JP2.5
- net CONVST: no longer JP2.1
- net CS: no longer JP2.4
- net GND: now also C13.2, C14.2, C19.2, C20.2, C21.2, C22.2, C23.2, C24.2, C25.2, C26.2, IC3.GND, IC4.GND, IC5.GND, JP1.2, JP4.2; no longer C13.-, C14.-
- net RESET: no longer JP2.2
- net SPI1_MISO: no longer JP2.6
- net SPI1_SCLK: no longer JP2.3
