File: Hardware/scanner.sch (EAGLE design)
At the start: 48 parts, among them IC2 FT232RL, IC3 MCP1703DB, IC4 MCP1703DB, IC5 MCP1703DB, U1 DAC8564IAPW, U2 AD7606BSTZ, X1 PN61729-S

Commit message: merging towards unity
Parts:
- removed C22, C23: (no value), resistor:C-EUC0805K
- removed D1: 1N4004, diode:1N4004
- removed IC2: FT232RL, ftdichip:FT232RL
- removed JP3: (no value), pinhead:PINHD-1X8
- removed JP4: (no value), pinhead:PINHD-1X3
- removed U$1: STM32F4-DISCOVERY, STM32F4-DISCOVERY:STM32F4-DISCOVERY
- removed X1: PN61729-S, con-berg:PN61729-S
- removed X2: (no value), con-subd:F15HDHS
- added AUX, CHANNEL_X, CHANNEL_Y, CHANNEL_Z: 1-227161-0, con-coax:1-227161-0
- added JP2: (no value), pinhead:PINHD-1X12
- added L1, L2, L3, L4: (no value), resistor:R-EU_M1206
- added R10, R11, R9: (no value), ptc-ntc:NTC644C
- added U$2: STM32F4-DISCOVERY, stm32full:STM32F4-DISCOVERY
- added X3: MSTBA10, con-phoenix-508:MSTBA10
- added X4: MSTBA4, con-phoenix-508:MSTBA4
- C10, C19, C21, C24: device resistor:C-EUC0805K -> resistor:C-EUC0805
- C12, C13, C18, C5, C6, C7: device resistor:C-EUC0805 -> resistor:C-EUC1206
- C20, C25, C26, C8, C9: device resistor:C-EUC0805K -> resistor:C-EUC1206
- IC5: value MCP1703DB -> 7812TV; device linear:MCP1703DB -> linear:7812TV
- JP1: device pinhead:PINHD-1X2 -> pinhead:PINHD-1X12
- U2: value AD7606BSTZ -> LTC1859CGPBF; device ad7606:AD7606BSTZ -> ltc1859:LTC1859CGPBF
Connections:
- removed net +15V: C25.1, D1.A, IC1P.V+, JP4.1, X2-14.F
- removed net -15V: C26.1, IC1P.V-, JP4.3, X2-15.F
- removed net BUSY: U$1.PA4, U2.BUSY
- removed net CS: U$1.PA3, U2.~CS
- removed net Q1-Q2_BUF: U2.V1, X2-1.F
- removed net Q1-Q4_BUF: U2.AGND, X2-3.F
- removed net Q1_BUF: U2.AGND_12, X2-9.F
- removed net Q2-Q3_BUF: U2.AGND_3, X2-13.F
- removed net Q2_BUF: U2.V3, X2-10.F
- removed net Q3_BUF: U2.V4, X2-11.F
- removed net Q4-Q3_BUF: U2.V2, X2-2.F
- removed net Q4_BUF: U2.AGND_13, X2-12.F
- removed net RESET: U$1.PA2, U2.RESET
- new net +12V: C18.1, C19.1, C26.1, IC1P.V+, IC5.VI, X4-4.1
- new net -12V: C20.1, C21.1, IC1P.V-, X4-1.1
- new net AGND: C3.2, C4.2, C7.2, C8.2, C9.2, L2.2, U2.AGND1, U2.AGND2, U2.AGND3, U2.COM, X3-10.1, X3-9.1
- new net AVCC: C3.1, C7.1, L1.2, U2.AVDD
- new net N$13: U2.CH7, X3-1.1
- new net N$14: IC1A.+IN, U1.VOUTB
- new net N$27: C11.1, C12.1, L3.2, U1.AVDD
- new net N$28: L4.2, R11.1
- new net N$30: C1.1, C5.1, R10.1, U2.OVDD
- new net N$4: C9.1, U2.VREF
- new net V+: C16.1, C24.1, C25.1, IC3.VI, IC4.VI, IC5.VO
- new net ~BUSY: U$2.PA4, U2.~BUSY
- net +3V3: now also IC4.VO, R10.2, R11.2; no longer C1.1, C12.1, C13.1, C14.1, C20.1, IC3.VO, U1.AVDD, U1.IO_VDD, U2.OS_2, U2.REF_SELECT, U2.VDRIVE, U2.~PAR/SER/BYTE_SEL, U2.~STBY
- net +5V: now also C17.1, IC3.VO, R9.2, U$2.5V, U$2.5V2; no longer C19.1, C2.1, C3.1, C4.1, C5.1, IC4.VO, U2.AVCC, U2.AVCC_2, U2.AVCC_3, U2.AVCC_4
- net CONVST: now also U$2.PA1, U2.CONVST; no longer U$1.PA1, U2.CONVST_A, U2.CONVST_B
- net GND: now also AUX.2, CHANNEL_X.2, CHANNEL_Y.2, CHANNEL_Z.2, JP1.6, L2.1, U$2.GND, U$2.GND1, U$2.GND2, U$2.GND3, U$2.GND4, U$2.GND5, U$2.GND6, U$2.GND7, U$2.GND8, U$2.GND9, U2.DGND, U2.~RD, X4-2.1, X4-3.1; no longer C22.2, C23.2, C3.2, C4.2, C7.2, C8.2, C9.2, IC2.GND, IC2.GND@1, IC2.GND@2, IC2.GND@A, IC2.TEST, JP1.2, JP3.2, JP3.4, JP3.6, JP3.8, JP4.2, U$1.GND, U$1.GND1, U$1.GND2, U$1.GND3, U$1.GND4, U$1.GND5, U2.AGND_10, U2.AGND_11, U2.AGND_14, U2.AGND_2, U2.AGND_4, U2.AGND_5, U2.AGND_6, U2.AGND_7, U2.AGND_8, U2.AGND_9, U2.DB0, U2.DB1, U2.DB10, U2.DB11, U2.DB12, U2.DB13, U2.DB15/BYTE_SEL, U2.DB2, U2.DB3, U2.DB4, U2.DB5, U2.DB6, U2.DB9, U2.OS_0, U2.OS_1, U2.RANGE, U2.REFGND, U2.REFGND_2, U2.V1GND, U2.V2GND, U2.V3GND, U2.V4GND, X1.4, X1.S1, X1.S2, X2-5.F, X2-6.F, X2-7.F, X2-8.F
- net N$1: now also U2.ADC+, U2.MUXOUT+; no longer C16.1, C18.1, IC2.VCC, X1.1
- net N$10: now also U2.CH4, X3-4.1; no longer C6.1, U2.REGCAP_2
- net N$11: now also U2.CH5, X3-3.1; no longer C17.1, IC2.3V3OUT, IC2.VCCIO
- net N$12: now also U2.CH6, X3-2.1; no longer C21.1, IC5.VO, JP1.1
- net N$15: now also IC1D.+IN, U1.VOUTC; no longer C10.1, U2.REFIN/REFOUT
- net N$16: now also U1.VOUTD; no longer U1.VOUTC
- net N$17: now also C10.1, U1.VREFH/VREFOUT; no longer IC1D.+IN, U1.VOUTD
- net N$18: now also CHANNEL_X.1, IC1B.OUT, R1.2; no longer C11.1, U1.VREFH/VREFOUT
- net N$19: now also IC1B.-IN, R1.1, R2.2; no longer IC1A.OUT, JP3.1, R1.2
- net N$2: now also U2.ADC-, U2.MUXOUT-; no longer IC2.USBDM, X1.2
- net N$20: now also CHANNEL_Y.1, IC1A.OUT, R3.1; no longer IC1A.-IN, R1.1, R2.2
- net N$21: now also IC1A.-IN, R3.2, R4.1; no longer IC1B.OUT, JP3.3, R3.1
- net N$22: now also C13.1, C14.1, L3.1, L4.1, U1.IO_VDD; no longer IC1B.-IN, R3.2, R4.1
- net N$23: now also CHANNEL_Z.1, IC1D.OUT; no longer IC1C.OUT, JP3.5
- net N$24: now also IC1D.-IN; no longer IC1C.-IN
- net N$25: now also AUX.1, IC1C.OUT; no longer IC1D.OUT, JP3.7
- net N$26: now also IC1C.-IN; no longer IC1D.-IN
- net N$29: now also C2.1, C6.1, L1.1, R9.1, U2.DVDD; no longer C22.1, C23.1, C24.1, D1.C, IC3.VI, IC4.VI, IC5.VI
- net N$3: now also IC1B.+IN, U1.VOUTA; no longer IC2.USBDP, X1.3
- net N$5: now also C4.1, C8.1, U2.REFCOMP; no longer IC1A.+IN, U1.VOUTA
- net N$6: now also U2.CH1, X3-7.1; no longer IC1B.+IN, U1.VOUTB
- net N$7: now also U2.CH0, X3-8.1; no longer C7.1, U2.REGCAP
- net N$8: now also U2.CH2, X3-6.1; no longer C8.1, U2.REFCAPB
- net N$9: now also U2.CH3, X3-5.1; no longer C9.1, U2.REFCAPA
- net SPI1_MISO: now also U$2.PA6, U2.SDO; no longer U$1.PA6, U2.DB7/DOUTA
- net SPI1_MOSI: now also U$2.PA7, U2.SDI; no longer U$1.PA7
- net SPI1_SCLK: now also U$2.PA5, U2.SCK; no longer U$1.PA5, U2.~RD/SCLK
- net SPI2_MISO: now also U$2.PB14; no longer U$1.PB14
- net SPI2_MOSI: now also U$2.PB15; no longer U$1.PB15
- net SPI2_SCLK: now also U$2.PB13; no longer U$1.PB13
- net USART3_RX: now also JP1.12, U$2.PD9; no longer IC2.TXD, U$1.PD9
- net USART3_TX: now also JP1.8, U$2.PD8; no longer IC2.RXD, U$1.PD8
- net ~SYNC: now also U$2.PB11; no longer U$1.PB11
Other:
- moved on the sheet: C1, C10, C11, C12, C13, C14, C15, C16, C17, C18, C19, C2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
